File: pcb/HabitReminderV2/HabitReminderV2.kicad_sch (KiCad schematic)
At the start: 11 parts, among them J1 USB_C_Receptacle_USB2.0, SW1 SW_Push, SW2 SW_Push, SW3 SW_Push, U1 ESP32-S3-WROOM-1, U2 LD1117S33TR_SOT223, U3 CP2102N-Axx-xQFN28

Commit message: schematic updates
Parts:
- added C1, C2: 22uF, symbol Device:C
- added C3, C4: C, symbol Device:C
- added SW4: BOOT_SW, symbol Switch:SW_Push
- added SW5: RST_SW, symbol Switch:SW_Push
Connections:
- net +3.3V: now also C1.1
- net GND: now also C1.2, C2.2, C3.1, C4.1, SW4.1, SW5.1
- net VBUS: now also C2.1
- net IO0: now reaches U1.27 (GPIO0/BOOT)
- net IO0: now also C3.2, SW4.2
- net EN: now reaches U1.3 (EN)
- net EN: now also C4.2, SW5.2
Other:
- moved on the sheet: J1, U2
